Commit message: Report the suspension joints' positions so RViz can draw the legs and wheels
The four suspension joints join ros2_control with state interfaces only (no command; gz_ros2_control 0.7.2 and later leave such joints alone), so the joint state broadcaster publishes them and robot_state_publisher places the legs and wheels.

File: src/agri_ugv_description/urdf/gazebo_control.xacro (robot description, xacro)
@@ -1,5 +1,8 @@
 <?xml version="1.0"?>
 <!-- ros2_control in Gazebo: each steering joint takes a position command,
-     each wheel joint a velocity command. The suspension stays passive. -->
+     each wheel joint a velocity command. The suspension stays passive: its joints only
+     report where they are (on /joint_states, so that robot_state_publisher can place the
+     legs and wheels, e.g. in RViz); joints without a command are left alone by
+     gz_ros2_control 0.7.2 and later. -->
 <robot xmlns:xacro="http://www.ros.org/wiki/xacro">
   <xacro:macro name="steer_joint_interface" params="prefix">
@@ -13,4 +16,10 @@
     <joint name="${prefix}_wheel_joint">
       <command_interface name="velocity"/>
+      <state_interface name="position"/>
+      <state_interface name="velocity"/>
+    </joint>
+  </xacro:macro>
+  <xacro:macro name="suspension_joint_interface" params="prefix">
+    <joint name="${prefix}_suspension_joint">
       <state_interface name="position"/>
       <state_interface name="velocity"/>
@@ -30,4 +39,8 @@
       <xacro:wheel_joint_interface prefix="rear_left"/>
       <xacro:wheel_joint_interface prefix="rear_right"/>
+      <xacro:suspension_joint_interface prefix="front_left"/>
+      <xacro:suspension_joint_interface prefix="front_right"/>
+      <xacro:suspension_joint_interface prefix="rear_left"/>
+      <xacro:suspension_joint_interface prefix="rear_right"/>
     </ros2_control>
     <!-- The Gazebo plugin that runs ros2_control inside the simulation -->
