Commit message: Add four wheel modules (steering, suspension, wheel) via xacro macro

File: src/agri_ugv_description/urdf/agri_ugv.urdf.xacro (robot description, xacro)
@@ -10,9 +10,22 @@
   <xacro:property name="box_top_z"       value="1.85"/>   <!-- above ground -->
   <xacro:property name="panel_thickness" value="0.02"/>
+  <xacro:property name="steer_z"         value="0.70"/>   <!-- steering motor height above ground (estimated) -->
+  <xacro:property name="susp_travel"     value="0.05"/>   <!-- +/- 5 cm, 0.10 m total (assumed) -->
+  <xacro:property name="steer_limit"     value="${pi/2}"/> <!-- +/- 90 degrees -->
   <!-- Derived values: computed, never typed twice -->
   <xacro:property name="box_height" value="${box_top_z - box_bottom_z}"/>
+  <xacro:property name="leg_length" value="${steer_z - wheel_radius}"/>
   <!-- ============ Colours for RViz ============ -->
   <material name="aluminium">
     <color rgba="0.75 0.75 0.78 1.0"/>
+  </material>
+  <material name="module_white">
+    <color rgba="0.95 0.95 0.95 1.0"/>
+  </material>
+  <material name="rubber">
+    <color rgba="0.15 0.15 0.15 1.0"/>
+  </material>
+  <material name="rim_red">
+    <color rgba="0.80 0.10 0.10 1.0"/>
   </material>
   <!-- ============ Reference points ============ -->
@@ -61,3 +74,74 @@
     <origin xyz="0 0 ${box_bottom_z - wheel_radius}" rpy="0 0 0"/>
   </joint>
+  <!-- ============ Wheel module: one corner ============ -->
+  <!-- prefix: module name, e.g. front_left
+       x_sign: +1 = front, -1 = rear
+       y_sign: +1 = left,  -1 = right -->
+  <xacro:macro name="wheel_module" params="prefix x_sign y_sign">
+    <!-- 1. Steering motor: turns everything below it around a vertical axis -->
+    <link name="${prefix}_steer_link">
+      <visual>
+        <geometry>
+          <box size="0.20 0.20 0.20"/>
+        </geometry>
+        <material name="module_white"/>
+      </visual>
+    </link>
+    <joint name="${prefix}_steer_joint" type="revolute">
+      <parent link="base_link"/>
+      <child link="${prefix}_steer_link"/>
+      <origin xyz="${x_sign*wheelbase/2} ${y_sign*track/2} ${steer_z - wheel_radius}" rpy="0 0 0"/>
+      <axis xyz="0 0 1"/>
+      <limit lower="${-steer_limit}" upper="${steer_limit}" effort="100" velocity="1.0"/>
+    </joint>
+    <!-- 2. Leg with suspension: slides up and down.
+         The leg is drawn beside the wheel, on the inner side. -->
+    <link name="${prefix}_leg_link">
+      <visual>
+        <origin xyz="0 ${-y_sign*(wheel_width/2 + 0.05)} ${-leg_length/2}" rpy="0 0 0"/>
+        <geometry>
+          <box size="0.10 0.06 ${leg_length}"/>
+        </geometry>
+        <material name="module_white"/>
+      </visual>
+    </link>
+    <joint name="${prefix}_suspension_joint" type="prismatic">
+      <parent link="${prefix}_steer_link"/>
+      <child link="${prefix}_leg_link"/>
+      <origin xyz="0 0 0" rpy="0 0 0"/>
+      <axis xyz="0 0 1"/>
+      <limit lower="${-susp_travel}" upper="${susp_travel}" effort="1000" velocity="0.5"/>
+    </joint>
+    <!-- 3. Wheel: spins around its axle (the y axis) -->
+    <link name="${prefix}_wheel_link">
+      <!-- Tyre. Cylinders stand upright by default, so roll 90 deg to lay the axle along y -->
+      <visual>
+        <origin xyz="0 0 0" rpy="${pi/2} 0 0"/>
+        <geometry>
+          <cylinder radius="${wheel_radius}" length="${wheel_width}"/>
+        </geometry>
+        <material name="rubber"/>
+      </visual>
+      <!-- Rim -->
+      <visual>
+        <origin xyz="0 0 0" rpy="${pi/2} 0 0"/>
+        <geometry>
+          <cylinder radius="${wheel_radius*0.5}" length="${wheel_width + 0.01}"/>
+        </geometry>
+        <material name="rim_red"/>
+      </visual>
+    </link>
+    <joint name="${prefix}_wheel_joint" type="continuous">
+      <parent link="${prefix}_leg_link"/>
+      <child link="${prefix}_wheel_link"/>
+      <!-- Wheel centre sits leg_length below the steering motor: exactly at axle height -->
+      <origin xyz="0 0 ${-leg_length}" rpy="0 0 0"/>
+      <axis xyz="0 1 0"/>
+    </joint>
+  </xacro:macro>
+  <!-- ============ The four corners ============ -->
+  <xacro:wheel_module prefix="front_left"  x_sign="1"  y_sign="1"/>
+  <xacro:wheel_module prefix="front_right" x_sign="1"  y_sign="-1"/>
+  <xacro:wheel_module prefix="rear_left"   x_sign="-1" y_sign="1"/>
+  <xacro:wheel_module prefix="rear_right"  x_sign="-1" y_sign="-1"/>
 </robot>

Commit message: Add mass, inertia and collision shapes; test total mass, centre of mass and tip-over angle

File: src/agri_ugv_description/urdf/agri_ugv.urdf.xacro (robot description, xacro)
@@ -1,4 +1,5 @@
 <?xml version="1.0"?>
 <robot name="agri_ugv" xmlns:xacro="http://www.ros.org/wiki/xacro">
+  <xacro:include filename="inertial_macros.xacro"/>
   <!-- ============ Dimensions (sources: docs/robot_spec.md) ============ -->
   <xacro:property name="track"           value="1.50"/>   <!-- left-right wheel spacing -->
@@ -13,4 +14,12 @@
   <xacro:property name="susp_travel"     value="0.05"/>   <!-- +/- 5 cm, 0.10 m total (assumed) -->
   <xacro:property name="steer_limit"     value="${pi/2}"/> <!-- +/- 90 degrees -->
+  <!-- ============ Masses (assumed; see docs/robot_spec.md) ============ -->
+  <xacro:property name="enclosure_mass"  value="100.0"/>  <!-- enclosure, sensors, computers -->
+  <xacro:property name="enclosure_com_z" value="1.40"/>   <!-- above ground -->
+  <xacro:property name="chassis_mass"    value="100.0"/>  <!-- frame and batteries -->
+  <xacro:property name="chassis_com_z"   value="0.80"/>   <!-- above ground -->
+  <xacro:property name="steer_mass"      value="4.0"/>    <!-- per module: steering motor -->
+  <xacro:property name="leg_mass"        value="6.0"/>    <!-- per module: leg, suspension, drive motor -->
+  <xacro:property name="wheel_mass"      value="10.0"/>   <!-- per module: wheel and tyre -->
   <!-- Derived values: computed, never typed twice -->
   <xacro:property name="box_height" value="${box_top_z - box_bottom_z}"/>
@@ -39,4 +48,13 @@
     <origin xyz="0 0 ${wheel_radius}" rpy="0 0 0"/>
   </joint>
+  <!-- ============ Chassis: frame and batteries (mass only, no visual) ============ -->
+  <link name="chassis">
+    <xacro:box_inertial mass="${chassis_mass}" x="${box_size}" y="${box_size}" z="0.20"/>
+  </link>
+  <joint name="chassis_joint" type="fixed">
+    <parent link="base_link"/>
+    <child link="chassis"/>
+    <origin xyz="0 0 ${chassis_com_z - wheel_radius}" rpy="0 0 0"/>
+  </joint>
   <!-- ============ Sensor enclosure ============ -->
   <!-- Roof plus left and right side panels. Front, rear and bottom are open,
@@ -51,4 +69,10 @@
       <material name="aluminium"/>
     </visual>
+    <collision>
+      <origin xyz="0 0 ${box_height - panel_thickness/2}" rpy="0 0 0"/>
+      <geometry>
+        <box size="${box_size} ${box_size} ${panel_thickness}"/>
+      </geometry>
+    </collision>
     <!-- Left side panel (+y) -->
     <visual>
@@ -59,4 +83,10 @@
       <material name="aluminium"/>
     </visual>
+    <collision>
+      <origin xyz="0 ${box_size/2 - panel_thickness/2} ${box_height/2}" rpy="0 0 0"/>
+      <geometry>
+        <box size="${box_size} ${panel_thickness} ${box_height}"/>
+      </geometry>
+    </collision>
     <!-- Right side panel (-y) -->
     <visual>
@@ -67,4 +97,13 @@
       <material name="aluminium"/>
     </visual>
+    <collision>
+      <origin xyz="0 ${-(box_size/2 - panel_thickness/2)} ${box_height/2}" rpy="0 0 0"/>
+      <geometry>
+        <box size="${box_size} ${panel_thickness} ${box_height}"/>
+      </geometry>
+    </collision>
+    <!-- Mass of the enclosure plus everything mounted in it -->
+    <xacro:box_inertial mass="${enclosure_mass}" x="${box_size}" y="${box_size}" z="${box_height}"
+                        xyz="0 0 ${enclosure_com_z - box_bottom_z}"/>
   </link>
   <joint name="enclosure_joint" type="fixed">
@@ -87,4 +126,5 @@
         <material name="module_white"/>
       </visual>
+      <xacro:box_inertial mass="${steer_mass}" x="0.20" y="0.20" z="0.20"/>
     </link>
     <joint name="${prefix}_steer_joint" type="revolute">
@@ -105,4 +145,6 @@
         <material name="module_white"/>
       </visual>
+      <xacro:box_inertial mass="${leg_mass}" x="0.10" y="0.06" z="${leg_length}"
+                          xyz="0 ${-y_sign*(wheel_width/2 + 0.05)} ${-leg_length/2}"/>
     </link>
     <joint name="${prefix}_suspension_joint" type="prismatic">
@@ -131,4 +173,13 @@
         <material name="rim_red"/>
       </visual>
+      <!-- The part that touches the ground -->
+      <collision>
+        <origin xyz="0 0 0" rpy="${pi/2} 0 0"/>
+        <geometry>
+          <cylinder radius="${wheel_radius}" length="${wheel_width}"/>
+        </geometry>
+      </collision>
+      <xacro:cylinder_inertial mass="${wheel_mass}" radius="${wheel_radius}" length="${wheel_width}"
+                               rpy="${pi/2} 0 0"/>
     </link>
     <joint name="${prefix}_wheel_joint" type="continuous">

Commit message: Add Gazebo package with flat world; passive suspension sized to rest at mid-travel

File: src/agri_ugv_description/urdf/agri_ugv.urdf.xacro (robot description, xacro)
@@ -22,4 +22,12 @@
   <xacro:property name="leg_mass"        value="6.0"/>    <!-- per module: leg, suspension, drive motor -->
   <xacro:property name="wheel_mass"      value="10.0"/>   <!-- per module: wheel and tyre -->
+  <!-- ============ Suspension: passive spring and damper per wheel ============ -->
+  <!-- Stiffness is chosen so the robot rests at mid-travel: each spring carries its
+       share of the sprung weight when compressed susp_travel from full extension. -->
+  <xacro:property name="gravity"               value="9.81"/>
+  <xacro:property name="susp_damping_ratio"    value="0.4"/>   <!-- assumed; 0.3-0.5 is typical -->
+  <xacro:property name="sprung_mass_per_wheel" value="${(enclosure_mass + chassis_mass + 4*steer_mass) / 4}"/>
+  <xacro:property name="susp_stiffness"        value="${sprung_mass_per_wheel * gravity / susp_travel}"/>
+  <xacro:property name="susp_damping"          value="${2 * susp_damping_ratio * sqrt(susp_stiffness * sprung_mass_per_wheel)}"/>
   <!-- Derived values: computed, never typed twice -->
   <xacro:property name="box_height" value="${box_top_z - box_bottom_z}"/>
@@ -154,5 +162,11 @@
       <axis xyz="0 0 1"/>
       <limit lower="${-susp_travel}" upper="${susp_travel}" effort="1000" velocity="0.5"/>
+      <dynamics damping="${susp_damping}" friction="0.0"/>
     </joint>
+    <!-- Spring: pushes the leg down, with zero force at full extension -->
+    <gazebo reference="${prefix}_suspension_joint">
+      <springReference>${-susp_travel}</springReference>
+      <springStiffness>${susp_stiffness}</springStiffness>
+    </gazebo>
     <!-- 3. Wheel: spins around its axle (the y axis) -->
     <link name="${prefix}_wheel_link">

Commit message: Add an IMU on the robot body (sensors.xacro, /imu)
100 Hz, no noise yet. At rest on the MuST-C field the accelerometer matches gravity predicted from the true tilt (pitch +0.71, roll -0.21 deg) to 0.1 mm/s2; |a| = 9.8000 (Gazebo's default gravity); orientation 0.000 deg from ground truth.

File: src/agri_ugv_description/urdf/agri_ugv.urdf.xacro (robot description, xacro)
@@ -4,4 +4,5 @@
   <xacro:include filename="gazebo_control.xacro"/>
   <xacro:include filename="soil.xacro"/>
+  <xacro:include filename="sensors.xacro"/>
   <!-- Path to the controller settings; empty = no ros2_control (e.g. RViz only) -->
   <xacro:arg name="controllers_file" default=""/>
@@ -216,4 +217,7 @@
   <xacro:wheel_module prefix="rear_left"   x_sign="-1" y_sign="1"/>
   <xacro:wheel_module prefix="rear_right"  x_sign="-1" y_sign="-1"/>
+  <!-- ============ Sensors (sensors.xacro) ============ -->
+  <xacro:property name="imu_height" value="0.90"/>  <!-- above ground, near the centre of mass -->
+  <xacro:imu_sensor z="${imu_height - wheel_radius}" rate="100"/>
     <!-- ============ ros2_control (only when a controllers file is given) ============ -->
   <xacro:if value="${'$(arg controllers_file)' != ''}">

Commit message: Add two roof GNSS antennas and align simulated GNSS with the UTM map
NavSat receivers 1.20 m apart, 1.90 m above ground, 10 Hz, no noise yet. Measured: with heading_deg 0 the fixes, converted through UTM, were 1.8 cm off and the antenna heading -1.50 deg (true +0.057): the UTM grid is turned 1.558 deg from true north here (meridian convergence). Read Gazebo's LOCAL2 conversion, set heading_deg = 1.558 and a 9-decimal origin: now 0.1 mm and +0.057 deg. Tilt lever arm visible: 0.71 deg pitch moves the front antenna 2.2 cm.

File: src/agri_ugv_description/urdf/agri_ugv.urdf.xacro (robot description, xacro)
@@ -220,4 +220,9 @@
   <xacro:property name="imu_height" value="0.90"/>  <!-- above ground, near the centre of mass -->
   <xacro:imu_sensor z="${imu_height - wheel_radius}" rate="100"/>
+  <xacro:property name="gnss_height"   value="1.90"/>  <!-- antennas 5 cm above the roof -->
+  <xacro:property name="gnss_baseline" value="1.20"/>  <!-- front-rear distance, gives the heading -->
+  <xacro:gnss_antenna name="front" x="${gnss_baseline/2}"  z="${gnss_height - wheel_radius}" rate="10"/>
+  <xacro:gnss_antenna name="rear"  x="${-gnss_baseline/2}" z="${gnss_height - wheel_radius}" rate="10"/>
+  <xacro:gnss_system/>
     <!-- ============ ros2_control (only when a controllers file is given) ============ -->
   <xacro:if value="${'$(arg controllers_file)' != ''}">

File: src/agri_ugv_description/urdf/sensors.xacro (robot description, xacro)
@@ -23,3 +23,28 @@
     </gazebo>
   </xacro:macro>
+  <!-- GNSS antenna: a NavSat receiver (no noise yet) publishing latitude, longitude and
+       altitude on /gnss/<name>/fix. Two antennas on the roof also give the heading. -->
+  <xacro:macro name="gnss_antenna" params="name x z rate">
+    <link name="gnss_${name}_link"/>
+    <joint name="gnss_${name}_joint" type="fixed">
+      <parent link="base_link"/>
+      <child link="gnss_${name}_link"/>
+      <origin xyz="${x} 0 ${z}" rpy="0 0 0"/>
+    </joint>
+    <gazebo reference="gnss_${name}_link">
+      <sensor name="gnss_${name}" type="navsat">
+        <always_on>true</always_on>
+        <update_rate>${rate}</update_rate>
+        <topic>/gnss/${name}/fix</topic>
+        <ignition_frame_id>gnss_${name}_link</ignition_frame_id>
+      </sensor>
+    </gazebo>
+  </xacro:macro>
+  <!-- Gazebo's NavSat system turns positions into latitude and longitude, using the
+       world's <spherical_coordinates> -->
+  <xacro:macro name="gnss_system">
+    <gazebo>
+      <plugin filename="ignition-gazebo-navsat-system" name="ignition::gazebo::systems::NavSat"/>
+    </gazebo>
+  </xacro:macro>
 </robot>

Commit message: Add the phenotyping payload (visual only) and move the IMU under the roof
After Esser et al. 2023: 20-camera dome aimed at the plant, two laser line scanners on the side panels (1.20 m, 50 deg from vertical), LED panels, curtains, computers, antenna pucks. No mass or collision added (still 280 kg, CoM 0.894 m). IMU now under the roof at the back like the real inertial unit; rest reading unchanged (diff 0.1 mm/s2). center_of_mass() now handles rotated joints instead of refusing them.

File: src/agri_ugv_description/urdf/agri_ugv.urdf.xacro (robot description, xacro)
@@ -5,4 +5,5 @@
   <xacro:include filename="soil.xacro"/>
   <xacro:include filename="sensors.xacro"/>
+  <xacro:include filename="payload.xacro"/>
   <!-- Path to the controller settings; empty = no ros2_control (e.g. RViz only) -->
   <xacro:arg name="controllers_file" default=""/>
@@ -218,6 +219,7 @@
   <xacro:wheel_module prefix="rear_right"  x_sign="-1" y_sign="-1"/>
   <!-- ============ Sensors (sensors.xacro) ============ -->
-  <xacro:property name="imu_height" value="0.90"/>  <!-- above ground, near the centre of mass -->
-  <xacro:imu_sensor z="${imu_height - wheel_radius}" rate="100"/>
+  <xacro:property name="imu_x"      value="-0.60"/> <!-- at the back, as on the real robot -->
+  <xacro:property name="imu_height" value="1.79"/>  <!-- above ground, just under the roof -->
+  <xacro:imu_sensor x="${imu_x}" z="${imu_height - wheel_radius}" rate="100"/>
   <xacro:property name="gnss_height"   value="1.90"/>  <!-- antennas 5 cm above the roof -->
   <xacro:property name="gnss_baseline" value="1.20"/>  <!-- front-rear distance, gives the heading -->
@@ -225,4 +227,6 @@
   <xacro:gnss_antenna name="rear"  x="${-gnss_baseline/2}" z="${gnss_height - wheel_radius}" rate="10"/>
   <xacro:gnss_system/>
+  <!-- ============ Phenotyping payload, visual only (payload.xacro) ============ -->
+  <xacro:payload roof_z="${box_top_z}"/>
     <!-- ============ ros2_control (only when a controllers file is given) ============ -->
   <xacro:if value="${'$(arg controllers_file)' != ''}">

File: src/agri_ugv_description/urdf/sensors.xacro (robot description, xacro)
@@ -3,11 +3,17 @@
      so every world gets them. -->
 <robot xmlns:xacro="http://www.ros.org/wiki/xacro">
-  <!-- IMU: accelerometer and gyroscope (no noise yet), published on /imu -->
-  <xacro:macro name="imu_sensor" params="z rate">
-    <link name="imu_link"/>
+  <!-- IMU: accelerometer and gyroscope (no noise yet), published on /imu. Like the real
+       robot's inertial unit, it sits under the roof at the back (Esser et al. 2023). -->
+  <xacro:macro name="imu_sensor" params="x z rate">
+    <link name="imu_link">
+      <visual>
+        <geometry><box size="0.16 0.12 0.06"/></geometry>
+        <material name="scanner_blue"/>
+      </visual>
+    </link>
     <joint name="imu_joint" type="fixed">
       <parent link="base_link"/>
       <child link="imu_link"/>
-      <origin xyz="0 0 ${z}" rpy="0 0 0"/>
+      <origin xyz="${x} 0 ${z}" rpy="0 0 0"/>
     </joint>
     <gazebo reference="imu_link">
@@ -26,5 +32,11 @@
        altitude on /gnss/<name>/fix. Two antennas on the roof also give the heading. -->
   <xacro:macro name="gnss_antenna" params="name x z rate">
-    <link name="gnss_${name}_link"/>
+    <link name="gnss_${name}_link">
+      <visual>                            <!-- antenna puck, its top at the phase centre -->
+        <origin xyz="0 0 -0.025" rpy="0 0 0"/>
+        <geometry><cylinder radius="0.07" length="0.05"/></geometry>
+        <material name="module_white"/>
+      </visual>
+    </link>
     <joint name="gnss_${name}_joint" type="fixed">
       <parent link="base_link"/>
