Commit message: Add a 3D LiDAR on a mast on the roof for driving
A spinning LiDAR like an Ouster OS0-64 (64 beams over +-45 deg, 1024 points per turn, 10 Hz, 0.3-50 m, 1 cm range noise) at the centre of the roof, 2.70 m above the ground. The robot of Esser et al. 2023 has none (it is driven by hand); an autonomous robot needs it to see the rows and anything in its way, all around because the passes go forwards and backwards. The mast lifts it high enough that its lowest beams pass over the roof edges ahead, behind and to the sides. Points on /lidar/points (PointCloud2, frame lidar_link); lidar:=false leaves the sensor and Gazebo's rendering system out; RViz view rviz/lidar.rviz.

Gazebo, robot standing at the start of soybean plot 188, 10 scans: 30208 of 65536 rays return a point (46.1 %; the upper half looks at the sky), 972 of them on the robot's roof corners, farthest 49.9 m. Plants: soybean 31-33 cm high (95 %; crop 30 cm, plants drawn 0.8-1.2 times that), 80-85 % of the soybean plant points within 10 cm of a crop row (44 % by chance); potato 42-43 cm, rows at chance level (closed canopy). Gazebo Fortress's GPU LiDAR renders every object with its own material, so it sees each leaf as its whole textured rectangle. Real-time factor 0.651 without the LiDAR, 0.527 with it (-19 %).

File: src/agri_ugv_description/urdf/agri_ugv.urdf.xacro (robot description, xacro)
@@ -10,4 +10,6 @@
   <!-- Soil profile in Gazebo: rigid (default, no slip model), firm, soft or wet (soil.xacro) -->
   <xacro:arg name="soil" default="rigid"/>
+  <!-- The 3D LiDAR on the roof (sensors.xacro); false leaves it out, e.g. to save rendering -->
+  <xacro:arg name="lidar" default="true"/>
   <!-- ============ Dimensions (sources: docs/robot_spec.md) ============ -->
   <xacro:property name="track"           value="1.50"/>   <!-- left-right wheel spacing -->
@@ -227,4 +229,10 @@
   <xacro:gnss_antenna name="rear"  x="${-gnss_baseline/2}" z="${gnss_height - wheel_radius}" rate="10"/>
   <xacro:gnss_system/>
+  <xacro:property name="lidar_height" value="2.70"/>  <!-- optical centre above ground, on a mast -->
+  <xacro:if value="$(arg lidar)">
+    <xacro:lidar_sensor z="${lidar_height - wheel_radius}" mast_bottom="${box_top_z - wheel_radius}"
+                        rate="10"/>
+    <xacro:rendering_system/>
+  </xacro:if>
   <!-- ============ Phenotyping payload, visual only (payload.xacro) ============ -->
   <xacro:payload roof_z="${box_top_z}"/>

File: src/agri_ugv_description/urdf/sensors.xacro (robot description, xacro)
@@ -90,3 +90,70 @@
     </gazebo>
   </xacro:macro>
+  <!-- 3D LiDAR for driving: a spinning LiDAR like an Ouster OS0-64 (64 beams over a 90 deg
+       vertical view, 1024 points per turn) on a mast on the roof. It is an addition to the
+       robot of Esser et al. 2023, which is driven by hand. The passes go forwards and
+       backwards, so it looks all around; the mast lifts it high enough that its lowest
+       beams (45 deg down) pass over the roof edges ahead, behind and to the sides. The point
+       cloud (sensor frame lidar_link) is published on /lidar/points; range noise assumed. -->
+  <xacro:macro name="lidar_sensor" params="z mast_bottom rate">
+    <link name="lidar_link">
+      <visual>                            <!-- sensor housing -->
+        <geometry><cylinder radius="0.043" length="0.07"/></geometry>
+        <material name="camera_black"/>
+      </visual>
+      <visual>                            <!-- mast, down to the roof -->
+        <origin xyz="0 0 ${-(z - mast_bottom) / 2}" rpy="0 0 0"/>
+        <geometry><cylinder radius="0.02" length="${z - mast_bottom}"/></geometry>
+        <material name="computer_grey"/>
+      </visual>
+    </link>
+    <joint name="lidar_joint" type="fixed">
+      <parent link="base_link"/>
+      <child link="lidar_link"/>
+      <origin xyz="0 0 ${z}" rpy="0 0 0"/>
+    </joint>
+    <gazebo reference="lidar_link">
+      <sensor name="lidar" type="gpu_lidar">
+        <always_on>true</always_on>
+        <update_rate>${rate}</update_rate>
+        <topic>/lidar</topic>
+        <ignition_frame_id>lidar_link</ignition_frame_id>
+        <visualize>false</visualize>
+        <lidar>
+          <scan>
+            <horizontal>
+              <samples>1024</samples>
+              <resolution>1</resolution>
+              <min_angle>${-pi}</min_angle>
+              <max_angle>${pi - 2 * pi / 1024}</max_angle>
+            </horizontal>
+            <vertical>
+              <samples>64</samples>
+              <resolution>1</resolution>
+              <min_angle>${-pi / 4}</min_angle>
+              <max_angle>${pi / 4}</max_angle>
+            </vertical>
+          </scan>
+          <range>
+            <min>0.3</min>
+            <max>50.0</max>
+            <resolution>0.001</resolution>
+          </range>
+          <noise>
+            <type>gaussian</type>
+            <mean>0.0</mean>
+            <stddev>0.01</stddev>
+          </noise>
+        </lidar>
+      </sensor>
+    </gazebo>
+  </xacro:macro>
+  <!-- Gazebo's Sensors system renders the camera-like sensors (the LiDAR) with Ogre 2 -->
+  <xacro:macro name="rendering_system">
+    <gazebo>
+      <plugin filename="ignition-gazebo-sensors-system" name="ignition::gazebo::systems::Sensors">
+        <render_engine>ogre2</render_engine>
+      </plugin>
+    </gazebo>
+  </xacro:macro>
 </robot>

Commit message: Add the two laser line scanners as sensors
Each side-panel scanner is a Gazebo GPU lidar with one fan of 300 rays over 35 deg across the robot (0.39-2 m, central ray 50 deg from vertical towards the far side), published as LaserScan on /scanners/left and /scanners/right. Launch arguments: scanners (default true) and scanner_rate (profiles per second, default 10). RViz setup: rviz/scanners.rviz.

At 30 profiles per second the simulation was overloaded: the wheel controller did not start in time and the robot did not move. At 10 per second it drives (real-time factor 0.53 together with the 3D LiDAR). Over sugar beet each scanner sees the ground from 0.10 to 0.92 m to the side and plant tops at 29-33 cm.

File: src/agri_ugv_description/urdf/agri_ugv.urdf.xacro (robot description, xacro)
@@ -12,4 +12,8 @@
   <!-- The 3D LiDAR on the roof (sensors.xacro); false leaves it out, e.g. to save rendering -->
   <xacro:arg name="lidar" default="true"/>
+  <!-- The two laser line scanners as sensors (sensors.xacro); false: visual only -->
+  <xacro:arg name="scanners" default="true"/>
+  <!-- their profiles per second; each one costs rendering time (the real ones: 200) -->
+  <xacro:arg name="scanner_rate" default="10"/>
   <!-- ============ Dimensions (sources: docs/robot_spec.md) ============ -->
   <xacro:property name="track"           value="1.50"/>   <!-- left-right wheel spacing -->
@@ -233,8 +237,17 @@
     <xacro:lidar_sensor z="${lidar_height - wheel_radius}" mast_bottom="${box_top_z - wheel_radius}"
                         rate="10"/>
+  </xacro:if>
+  <!-- ============ Phenotyping payload (payload.xacro) ============ -->
+  <xacro:payload roof_z="${box_top_z}"/>
+  <!-- the line scanners measure: 300 points over 35 deg each, scanner_rate per second -->
+  <xacro:if value="$(arg scanners)">
+    <xacro:line_scanner_sensor side="left" rate="$(arg scanner_rate)" samples="300"
+                               fan="${radians(35)}"/>
+    <xacro:line_scanner_sensor side="right" rate="$(arg scanner_rate)" samples="300"
+                               fan="${radians(35)}"/>
+  </xacro:if>
+  <xacro:if value="${'$(arg lidar)' in ('true', '1') or '$(arg scanners)' in ('true', '1')}">
     <xacro:rendering_system/>
   </xacro:if>
-  <!-- ============ Phenotyping payload, visual only (payload.xacro) ============ -->
-  <xacro:payload roof_z="${box_top_z}"/>
     <!-- ============ ros2_control (only when a controllers file is given) ============ -->
   <xacro:if value="${'$(arg controllers_file)' != ''}">

File: src/agri_ugv_description/urdf/sensors.xacro (robot description, xacro)
@@ -149,5 +149,56 @@
     </gazebo>
   </xacro:macro>
-  <!-- Gazebo's Sensors system renders the camera-like sensors (the LiDAR) with Ogre 2 -->
+  <!-- Laser line scanner (sensor): a fan of 'samples' rays, 'fan' wide, in the plane
+       across the robot that holds the scanner's central ray (link line_scanner_<side>_link,
+       payload.xacro: 50 deg from vertical, towards the middle). Like the robot's LMI Gocator
+       2490 scanners (Esser et al. 2023): range 0.39-2 m; the fan width, the noise and the
+       profile rate (the real one: 200 per second) are assumed, the rate much lower: each
+       profile costs rendering time. Each profile is published on /scanners/<side> (LaserScan) in the
+       frame line_scanner_<side>_beam_link: x along the central ray, the fan in its x-y
+       plane. Driving along the rows, the profiles add up to the plants' 3D shape. -->
+  <xacro:macro name="line_scanner_sensor" params="side rate samples fan">
+    <link name="line_scanner_${side}_beam_link"/>
+    <joint name="line_scanner_${side}_beam_joint" type="fixed">
+      <parent link="line_scanner_${side}_link"/>
+      <child link="line_scanner_${side}_beam_link"/>
+      <origin xyz="0 0 0" rpy="${pi / 2} 0 0"/>
+    </joint>
+    <gazebo reference="line_scanner_${side}_beam_link">
+      <sensor name="line_scanner_${side}" type="gpu_lidar">
+        <always_on>true</always_on>
+        <update_rate>${rate}</update_rate>
+        <topic>/scanners/${side}</topic>
+        <ignition_frame_id>line_scanner_${side}_beam_link</ignition_frame_id>
+        <visualize>false</visualize>
+        <lidar>
+          <scan>
+            <horizontal>
+              <samples>${samples}</samples>
+              <resolution>1</resolution>
+              <min_angle>${-fan / 2}</min_angle>
+              <max_angle>${fan / 2}</max_angle>
+            </horizontal>
+            <vertical>
+              <samples>1</samples>
+              <resolution>1</resolution>
+              <min_angle>0</min_angle>
+              <max_angle>0</max_angle>
+            </vertical>
+          </scan>
+          <range>
+            <min>0.39</min>
+            <max>2.0</max>
+            <resolution>0.0001</resolution>
+          </range>
+          <noise>
+            <type>gaussian</type>
+            <mean>0.0</mean>
+            <stddev>0.0005</stddev>
+          </noise>
+        </lidar>
+      </sensor>
+    </gazebo>
+  </xacro:macro>
+  <!-- Gazebo's Sensors system renders the camera-like sensors (LiDAR, line scanners) with Ogre 2 -->
   <xacro:macro name="rendering_system">
     <gazebo>

Commit message: Let the dome cameras take pictures
cameras:=top turns the 4 cameras of the dome's top ring into Gazebo cameras (640 x 480 pixels, 60 deg wide, 2 pictures per second, taken just in front of the lens), cameras:=all all 20; the default stays none. The pictures are published on /cameras/dome_<i>/image, with camera_info.

Plot 198, the 4 top cameras while driving: 2.0 pictures per simulated second each, plants on about half of every picture; real-time factor 0.49 (0.63-0.66 without cameras). The plant under the robot is in the shade of the roof (mean brightness 37 of 255).

File: src/agri_ugv_description/urdf/agri_ugv.urdf.xacro (robot description, xacro)
@@ -16,4 +16,9 @@
   <!-- their profiles per second; each one costs rendering time (the real ones: 200) -->
   <xacro:arg name="scanner_rate" default="10"/>
+  <!-- The dome cameras as sensors (sensors.xacro): none (visual only), top (the 4 of the top
+       ring, looking down at the plant) or all 20; each image costs rendering time -->
+  <xacro:arg name="cameras" default="none"/>
+  <!-- their images per second -->
+  <xacro:arg name="camera_rate" default="2"/>
   <!-- ============ Dimensions (sources: docs/robot_spec.md) ============ -->
   <xacro:property name="track"           value="1.50"/>   <!-- left-right wheel spacing -->
@@ -247,5 +252,15 @@
                                fan="${radians(35)}"/>
   </xacro:if>
-  <xacro:if value="${'$(arg lidar)' in ('true', '1') or '$(arg scanners)' in ('true', '1')}">
+  <!-- the cameras: 640 x 480 pixels, 60 deg wide (assumed lens) -->
+  <xacro:if value="${'$(arg cameras)' == 'top'}">
+    <xacro:dome_camera_sensors first="16" last="19" rate="$(arg camera_rate)" width="640"
+                               height="480" fov="${radians(60)}"/>
+  </xacro:if>
+  <xacro:if value="${'$(arg cameras)' == 'all'}">
+    <xacro:dome_camera_sensors first="0" last="19" rate="$(arg camera_rate)" width="640"
+                               height="480" fov="${radians(60)}"/>
+  </xacro:if>
+  <xacro:if value="${'$(arg lidar)' in ('true', '1') or '$(arg scanners)' in ('true', '1')
+                     or '$(arg cameras)' != 'none'}">
     <xacro:rendering_system/>
   </xacro:if>

File: src/agri_ugv_description/urdf/sensors.xacro (robot description, xacro)
@@ -200,5 +200,55 @@
     </gazebo>
   </xacro:macro>
-  <!-- Gazebo's Sensors system renders the camera-like sensors (LiDAR, line scanners) with Ogre 2 -->
+  <!-- Dome camera (sensor): one of the 20 cameras of the dome (payload.xacro), looking along
+       +x of dome_camera_<index>_link at the plant under the robot. The real ones are Nikon Z7
+       (45 megapixels, Esser et al. 2023); here a small image, a few per second, assumed lens:
+       every image renders the plants. The image is taken just in front of the lens, from
+       dome_camera_<index>_optical_link (x forward, as the camera link), and published on
+       /cameras/dome_<index>/image, its calibration on /cameras/dome_<index>/camera_info. -->
+  <xacro:macro name="dome_camera_sensor" params="index rate width height fov">
+    <link name="dome_camera_${index}_optical_link"/>
+    <joint name="dome_camera_${index}_optical_joint" type="fixed">
+      <parent link="dome_camera_${index}_link"/>
+      <child link="dome_camera_${index}_optical_link"/>
+      <origin xyz="0.095 0 0" rpy="0 0 0"/>
+    </joint>
+    <gazebo reference="dome_camera_${index}_optical_link">
+      <sensor name="dome_camera_${index}" type="camera">
+        <always_on>true</always_on>
+        <update_rate>${rate}</update_rate>
+        <topic>/cameras/dome_${index}/image</topic>
+        <ignition_frame_id>dome_camera_${index}_optical_link</ignition_frame_id>
+        <visualize>false</visualize>
+        <camera>
+          <horizontal_fov>${fov}</horizontal_fov>
+          <image>
+            <width>${width}</width>
+            <height>${height}</height>
+            <format>R8G8B8</format>
+          </image>
+          <clip>
+            <near>0.05</near>
+            <far>10.0</far>
+          </clip>
+          <noise>
+            <type>gaussian</type>
+            <mean>0.0</mean>
+            <stddev>0.007</stddev>
+          </noise>
+        </camera>
+      </sensor>
+    </gazebo>
+  </xacro:macro>
+  <!-- the dome cameras first..last (indices) as sensors -->
+  <xacro:macro name="dome_camera_sensors" params="first last rate width height fov">
+    <xacro:dome_camera_sensor index="${first}" rate="${rate}" width="${width}"
+                              height="${height}" fov="${fov}"/>
+    <xacro:if value="${first &lt; last}">
+      <xacro:dome_camera_sensors first="${first + 1}" last="${last}" rate="${rate}"
+                                 width="${width}" height="${height}" fov="${fov}"/>
+    </xacro:if>
+  </xacro:macro>
+  <!-- Gazebo's Sensors system renders the camera-like sensors (LiDAR, line scanners, cameras)
+       with Ogre 2 -->
   <xacro:macro name="rendering_system">
     <gazebo>

Commit message: Let the dome cameras measure depth when asked
camera_depth:=true makes the dome cameras RGB-D cameras: each also publishes /cameras/dome_<i>/depth_image (metres, 32FC1), for 3D reconstruction from one stop. Passed through sim, mission and survey launch files; default false.

File: src/agri_ugv_description/urdf/agri_ugv.urdf.xacro (robot description, xacro)
@@ -21,4 +21,6 @@
   <!-- their images per second -->
   <xacro:arg name="camera_rate" default="2"/>
+  <!-- true: the dome cameras also measure depth (RGB-D cameras, for 3D reconstruction) -->
+  <xacro:arg name="camera_depth" default="false"/>
   <!-- ============ Dimensions (sources: docs/robot_spec.md) ============ -->
   <xacro:property name="track"           value="1.50"/>   <!-- left-right wheel spacing -->
@@ -255,9 +257,9 @@
   <xacro:if value="${'$(arg cameras)' == 'top'}">
     <xacro:dome_camera_sensors first="16" last="19" rate="$(arg camera_rate)" width="640"
-                               height="480" fov="${radians(60)}"/>
+                               height="480" fov="${radians(60)}" depth="$(arg camera_depth)"/>
   </xacro:if>
   <xacro:if value="${'$(arg cameras)' == 'all'}">
     <xacro:dome_camera_sensors first="0" last="19" rate="$(arg camera_rate)" width="640"
-                               height="480" fov="${radians(60)}"/>
+                               height="480" fov="${radians(60)}" depth="$(arg camera_depth)"/>
   </xacro:if>
   <xacro:if value="${'$(arg lidar)' in ('true', '1') or '$(arg scanners)' in ('true', '1')

File: src/agri_ugv_description/urdf/sensors.xacro (robot description, xacro)
@@ -205,6 +205,9 @@
        every image renders the plants. The image is taken just in front of the lens, from
        dome_camera_<index>_optical_link (x forward, as the camera link), and published on
-       /cameras/dome_<index>/image, its calibration on /cameras/dome_<index>/camera_info. -->
-  <xacro:macro name="dome_camera_sensor" params="index rate width height fov">
+       /cameras/dome_<index>/image, its calibration on /cameras/dome_<index>/camera_info.
+       With depth, the camera also measures each pixel's depth (an RGB-D camera; the real
+       robot gets depth by matching its cameras' pictures): /cameras/dome_<index>/depth_image,
+       metres along the view (32FC1). -->
+  <xacro:macro name="dome_camera_sensor" params="index rate width height fov depth:=false">
     <link name="dome_camera_${index}_optical_link"/>
     <joint name="dome_camera_${index}_optical_joint" type="fixed">
@@ -214,8 +217,8 @@
     </joint>
     <gazebo reference="dome_camera_${index}_optical_link">
-      <sensor name="dome_camera_${index}" type="camera">
-        <always_on>true</always_on>
-        <update_rate>${rate}</update_rate>
-        <topic>/cameras/dome_${index}/image</topic>
+      <sensor name="dome_camera_${index}" type="${'rgbd_camera' if depth else 'camera'}">
+        <always_on>true</always_on>
+        <update_rate>${rate}</update_rate>
+        <topic>/cameras/dome_${index}${'' if depth else '/image'}</topic>
         <ignition_frame_id>dome_camera_${index}_optical_link</ignition_frame_id>
         <visualize>false</visualize>
@@ -241,10 +244,11 @@
   </xacro:macro>
   <!-- the dome cameras first..last (indices) as sensors -->
-  <xacro:macro name="dome_camera_sensors" params="first last rate width height fov">
+  <xacro:macro name="dome_camera_sensors" params="first last rate width height fov depth:=false">
     <xacro:dome_camera_sensor index="${first}" rate="${rate}" width="${width}"
-                              height="${height}" fov="${fov}"/>
+                              height="${height}" fov="${fov}" depth="${depth}"/>
     <xacro:if value="${first &lt; last}">
       <xacro:dome_camera_sensors first="${first + 1}" last="${last}" rate="${rate}"
-                                 width="${width}" height="${height}" fov="${fov}"/>
+                                 width="${width}" height="${height}" fov="${fov}"
+                                 depth="${depth}"/>
     </xacro:if>
   </xacro:macro>

Commit message: Let a model mount extra hardware with its own controllers on the robot

File: src/agri_ugv_description/urdf/agri_ugv.urdf.xacro (robot description, xacro)
@@ -8,4 +8,7 @@
   <!-- Path to the controller settings; empty = no ros2_control (e.g. RViz only) -->
   <xacro:arg name="controllers_file" default=""/>
+  <!-- A second controller settings file, for hardware mounted on the robot that has its own
+       ros2_control joints (e.g. an arm); empty = none (gazebo_control.xacro) -->
+  <xacro:arg name="extra_controllers_file" default=""/>
   <!-- Soil profile in Gazebo: rigid (default, no slip model), firm, soft or wet (soil.xacro) -->
   <xacro:arg name="soil" default="rigid"/>
@@ -269,5 +272,6 @@
     <!-- ============ ros2_control (only when a controllers file is given) ============ -->
   <xacro:if value="${'$(arg controllers_file)' != ''}">
-    <xacro:gazebo_control controllers_file="$(arg controllers_file)"/>
+    <xacro:gazebo_control controllers_file="$(arg controllers_file)"
+                          extra_controllers_file="$(arg extra_controllers_file)"/>
     <xacro:if value="${'$(arg soil)' != 'rigid'}">
       <xacro:soil_model soil="$(arg soil)"/>

File: src/agri_ugv_description/urdf/gazebo_control.xacro (robot description, xacro)
@@ -26,5 +26,8 @@
     </joint>
   </xacro:macro>
-  <xacro:macro name="gazebo_control" params="controllers_file">
+  <!-- extra_controllers_file: settings of the controllers of hardware mounted on the robot
+       (e.g. an arm with its own ros2_control joints); empty: none. Both files go to the
+       same controller manager, so one /joint_states covers all joints. -->
+  <xacro:macro name="gazebo_control" params="controllers_file extra_controllers_file:=''">
     <ros2_control name="GazeboSimSystem" type="system">
       <hardware>
@@ -49,4 +52,7 @@
               name="gz_ros2_control::GazeboSimROS2ControlPlugin">
         <parameters>${controllers_file}</parameters>
+        <xacro:if value="${extra_controllers_file != ''}">
+          <parameters>${extra_controllers_file}</parameters>
+        </xacro:if>
       </plugin>
     </gazebo>
